Commit message: add camera

File: ua_ros_p3dx/p3dx_description/urdf/pioneer3dx.xacro (robot description, xacro)
@@ -230,3 +230,55 @@
 		<child link="lms100" />
 	</joint>
+	<link name="camera_link">
+		<inertial>
+			<mass value="1e-5" />
+			<origin xyz="0 0 0" rpy="0 0 0" />
+			<inertia ixx="1e-6" ixy="0" ixz="0" iyy="1e-6" iyz="0" izz="1e-6" />
+		</inertial>
+		<visual>
+			<origin xyz="0 0 0" rpy="0 0 0" />
+			<geometry>
+				<mesh filename="package://p3dx_description/meshes/kinect.dae" />
+			</geometry>
+		</visual>
+		<collision>
+			<origin xyz="0 0 0" rpy="0 0 0" />
+			<geometry>
+				<box size="0.1 0.1 0.1" />
+			</geometry>
+		</collision>
+	</link>
+	<joint name="camera_joint" type="fixed">
+		<origin xyz="0 0 0.3" rpy="0 0 0" />
+		<parent link="base_link" />
+		<child link="camera_link" />
+	</joint>
+	<joint name="camera_depth_joint" type="fixed">
+		<origin xyz="0 0.028 0" rpy="0 0 0" />
+		<parent link="camera_link" />
+		<child link="camera_depth_frame" />
+	</joint>
+	<link name="camera_depth_frame">
+	<inertial>
+		<mass value="0.0001" />
+		<origin xyz="0 0 0" />
+		<inertia ixx="0.0001" ixy="0.0" ixz="0.0"
+				iyy="0.0001" iyz="0.0"
+				izz="0.0001" />
+	</inertial>
+	</link>
+	<joint name="depth_optical_joint" type="fixed">
+		<origin xyz="0 0 0" rpy="${-M_PI/2} 0 ${-M_PI/2}" />
+		<parent link="camera_depth_frame" />
+		<child link="camera_depth_optical_frame" />
+	</joint>
+	<link name="camera_depth_optical_frame">
+		<inertial>
+			<mass value="0.0001" />
+			<origin xyz="0 0 0" />
+			<inertia ixx="0.0001" ixy="0.0" ixz="0.0"
+				iyy="0.0001" iyz="0.0"
+				izz="0.0001" />
+		</inertial>
+	</link>
 </robot>

Commit message: update xacro and launches

File: ua_ros_p3dx/p3dx_description/urdf/pioneer3dx.xacro (robot description, xacro)
@@ -250,5 +250,5 @@
 	</link>
 	<joint name="camera_joint" type="fixed">
-		<origin xyz="0 0 0.3" rpy="0 0 0" />
+		<origin xyz="0.11 0 0.49" rpy="0 0 0" />
 		<parent link="base_link" />
 		<child link="camera_link" />

Commit message: Add camera to URDF

File: ua_ros_p3dx/p3dx_description/urdf/pioneer3dx.xacro (robot description, xacro)
@@ -163,5 +163,5 @@
 		</visual>
 		<collision>
-			<origin xyz="0 0 0" rpy="${-3.1415927/2.0} 0 0" />
+			<origin xyz="0 0 0" rpy="-1.5707 0 0" />
 			<geometry>
 				<cylinder radius="0.0375" length="0.01" />
@@ -205,5 +205,5 @@
 	</joint>
 	<!-- lms100 laser -->
-	<link name="lms100">
+	<link name="laser">
 		<inertial>
 			<mass value="1e-5" />
@@ -224,9 +224,9 @@
 		</collision>
 	</link>
-	<joint name="lms100_joint" type="fixed">
+	<joint name="laser_joint" type="fixed">
 		<axis xyz="0 1 0" />
 		<origin xyz="0.16 0 0.15" rpy="0 0 0" />
 		<parent link="base_link" />
-		<child link="lms100" />
+		<child link="laser" />
 	</joint>
 	<link name="camera_link">
@@ -269,5 +269,5 @@
 	</link>
 	<joint name="depth_optical_joint" type="fixed">
-		<origin xyz="0 0 0" rpy="${-M_PI/2} 0 ${-M_PI/2}" />
+		<origin xyz="0 0 0" rpy="-1.5707 0 -1.5707" />
 		<parent link="camera_depth_frame" />
 		<child link="camera_depth_optical_frame" />

File: ua_ros_p3dx/p3dx_description/urdf/pioneer3dx_wheel.xacro (robot description, xacro)
@@ -39,5 +39,5 @@
 			</visual>
 			<collision>
-				<origin xyz="0 0 0" rpy="${-3.1415927/2} 0 0" />
+				<origin xyz="0 0 0" rpy="-1.5707 0 0" />
 				<geometry>
 					<!--<mesh filename="package://p3dx_description/meshes/${suffix}_wheel.stl"/> -->
